File: USART_BoSL_Bus/USART_BoSL_Bus/USART_BoSL_Bus.sch (KiCad schematic (older format))
At the start: 8 parts

Commit message: added BOM for interconnect added layout for interconnect
Parts:
- J1: renamed from J?; footprint (none) -> Connector_RJ:RJ12_Amphenol_54601
- J2: renamed from J?; footprint Connector_PinSocket_2.54mm:PinSocket_1x08_P2.54mm_Vertical -> Connector_PinSocket_2.54mm:PinSocket_1x06_P2.54mm_Vertical
- gave numbers to parts that had none: 6
Connections:
- net labels removed: 3V3
- wire segments 94 -> 49
Other:
- note removed: "BoSL"
- note removed: "High - Z"
- note removed: "Low - Z"
- note removed: "RS-485"
- note removed: "Sensor"
- moved on the sheet: J2
